Commit message: Motor Driver

File: ros_ws/src/chitti_description/urdf/chitti.urdf.xacro (robot description, xacro)
@@ -125,3 +125,47 @@
     <origin xyz="0 0 ${base_height/2}" rpy="0 0 0"/>
   </joint>
+  <!-- ═══════════════════════════════════════
+       ROS2_CONTROL  –  Cytron MDD10A Hardware Interface
+       GPIO pin numbers are PLACEHOLDERS – update to your wiring!
+  ═══════════════════════════════════════ -->
+  <ros2_control name="chitti_hardware" type="system">
+    <hardware>
+      <plugin>chitti_control/CytronHardwareInterface</plugin>
+      <!-- Motor Driver 1 – Channel A: Front Left -->
+      <param name="fl_pwm_pin">12</param>
+      <param name="fl_dir_pin">5</param>
+      <!-- Motor Driver 1 – Channel B: Rear Left -->
+      <param name="rl_pwm_pin">13</param>
+      <param name="rl_dir_pin">6</param>
+      <!-- Motor Driver 2 – Channel A: Front Right -->
+      <param name="fr_pwm_pin">18</param>
+      <param name="fr_dir_pin">16</param>
+      <!-- Motor Driver 2 – Channel B: Rear Right -->
+      <param name="rr_pwm_pin">19</param>
+      <param name="rr_dir_pin">20</param>
+      <!-- Wheel physical parameters -->
+      <param name="wheel_radius">0.05</param>
+      <param name="max_motor_rpm">200</param>
+    </hardware>
+    <joint name="front_left_wheel_joint">
+      <command_interface name="velocity"/>
+      <state_interface name="position"/>
+      <state_interface name="velocity"/>
+    </joint>
+    <joint name="front_right_wheel_joint">
+      <command_interface name="velocity"/>
+      <state_interface name="position"/>
+      <state_interface name="velocity"/>
+    </joint>
+    <joint name="rear_left_wheel_joint">
+      <command_interface name="velocity"/>
+      <state_interface name="position"/>
+      <state_interface name="velocity"/>
+    </joint>
+    <joint name="rear_right_wheel_joint">
+      <command_interface name="velocity"/>
+      <state_interface name="position"/>
+      <state_interface name="velocity"/>
+    </joint>
+  </ros2_control>
 </robot>
